File: electronics/ServoBoard.sch (KiCad schematic (older format))
At the start: 8 parts, among them K1 Left Servo, K2 Right Servo, P1 Pi GPIO Header, P2 CONN_2, U1 7805

Commit message: Gerber Files
Parts:
- added P3, P4, P5, P6: CONNECTOR, ~, symbol CONNECTOR
Connections:
- no-connect marks 35 -> 39
Changed lines of the file:
@@
 Sheet 1 1
 Title "Robot Turtle Servo Board"
-Date "2 jan 2015"
+Date "3 jan 2015"
 Rev "0.01"
 Comp ""
@@
 $EndComp
 $Comp
-L +6V #PWR01
+L +6V #PWR1
 U 1 1 54A6D96E
 P 1400 1550
-F 0 "#PWR01" H 1400 1680 20  0001 C CNN
+F 0 "#PWR1" H 1400 1680 20  0001 C CNN
 F 1 "+6V" H 1400 1650 30  0000 C CNN
 F 2 "" H 1400 1550 60  0000 C CNN
@@
 $EndComp
 $Comp
-L GND #PWR02
+L GND #PWR2
 U 1 1 54A6DDCB
 P 1400 3050
-F 0 "#PWR02" H 1400 3050 30  0001 C CNN
+F 0 "#PWR2" H 1400 3050 30  0001 C CNN
 F 1 "GND" H 1400 2980 30  0001 C CNN
 F 2 "" H 1400 3050 60  0000 C CNN
@@
 Connection ~ 2700 4250
 $Comp
-L PWR_FLAG #FLG03
+L PWR_FLAG #FLG2
 U 1 1 54A6E288
 P 1050 1550
-F 0 "#FLG03" H 1050 1645 30  0001 C CNN
+F 0 "#FLG2" H 1050 1645 30  0001 C CNN
 F 1 "PWR_FLAG" H 1050 1730 30  0000 C CNN
 F 2 "" H 1050 1550 60  0000 C CNN
@@
 $EndComp
 $Comp
-L PWR_FLAG #FLG04
+L PWR_FLAG #FLG1
 U 1 1 54A6E297
 P 1000 2900
-F 0 "#FLG04" H 1000 2995 30  0001 C CNN
+F 0 "#FLG1" H 1000 2995 30  0001 C CNN
 F 1 "PWR_FLAG" H 1000 3080 30  0000 C CNN
 F 2 "" H 1000 2900 60  0000 C CNN
@@
 Wire Wire Line
 	1550 2350 1550 2400
+$Comp
+L CONNECTOR P3
+U 1 1 54A791F4
+P 1150 4900
+F 0 "P3" H 1500 5000 70  0000 C CNN
+F 1 "CONNECTOR" H 1500 4800 70  0000 C CNN
+F 2 "~" H 1150 4900 60  0000 C CNN
+F 3 "~" H 1150 4900 60  0000 C CNN
+	1    1150 4900
+	1    0    0    -1
+$EndComp
+$Comp
+L CONNECTOR P5
+U 1 1 54A79203
+P 2250 4900
+F 0 "P5" H 2600 5000 70  0000 C CNN
+F 1 "CONNECTOR" H 2600 4800 70  0000 C CNN
+F 2 "~" H 2250 4900 60  0000 C CNN
+F 3 "~" H 2250 4900 60  0000 C CNN
+	1    2250 4900
+	1    0    0    -1
+$EndComp
+$Comp
+L CONNECTOR P4
+U 1 1 54A79212
+P 1350 5400
+F 0 "P4" H 1700 5500 70  0000 C CNN
+F 1 "CONNECTOR" H 1700 5300 70  0000 C CNN
+F 2 "~" H 1350 5400 60  0000 C CNN
+F 3 "~" H 1350 5400 60  0000 C CNN
+	1    1350 5400
+	1    0    0    -1
+$EndComp
+$Comp
+L CONNECTOR P6
+U 1 1 54A79221
+P 2600 5400
+F 0 "P6" H 2950 5500 70  0000 C CNN
+F 1 "CONNECTOR" H 2950 5300 70  0000 C CNN
+F 2 "~" H 2600 5400 60  0000 C CNN
+F 3 "~" H 2600 5400 60  0000 C CNN
+	1    2600 5400
+	1    0    0    -1
+$EndComp
+NoConn ~ 2600 5400
+NoConn ~ 2250 4900
+NoConn ~ 1350 5400
+NoConn ~ 1150 4900
 $EndSCHEMATC

Commit message: Added 2nd connector for power, may be a bit too small
Parts:
- added P7: CONN_2, symbol CONN_2
Connections:
- net +6V: now also P7.2 (PM); no longer P2.2 (PM)
- new net: P2.2 (PM), P7.1 (P1)
Changed lines of the file:
@@
 Sheet 1 1
 Title "Robot Turtle Servo Board"
-Date "3 jan 2015"
+Date "4 jan 2015"
 Rev "0.01"
 Comp ""
@@
 $EndComp
 Wire Wire Line
-	1000 2150 1000 1650
-Wire Wire Line
 	1200 2800 1550 2800
 Connection ~ 1400 2900
@@
 NoConn ~ 1350 5400
 NoConn ~ 1150 4900
+$Comp
+L CONN_2 P7
+U 1 1 54A8EE48
+P 650 1850
+F 0 "P7" V 600 1850 40  0000 C CNN
+F 1 "CONN_2" V 700 1850 40  0000 C CNN
+F 2 "" H 650 1850 60  0000 C CNN
+F 3 "" H 650 1850 60  0000 C CNN
+	1    650  1850
+	-1   0    0    1
+$EndComp
+Wire Wire Line
+	1000 1650 1000 1750
+Wire Wire Line
+	1000 1950 1000 2150
 $EndSCHEMATC
